Commit message: all transformation are published by robot_state_publisher. Updated urdf file.

File: geduino/urdf/geduino.urdf (robot description, URDF)
Before this commit: robot geduino, 1 links, 0 joints
Links:
- added link base_camera
- added link base_imu
- added link base_laser; visual cylinder length=0.06 radius=0.035
Joints:
- added joint base_link_to_base_camera: type fixed, parent base_link, child base_camera, origin xyz=0 0 0 rpy=0 0 0
- added joint base_link_to_base_imu: type fixed, parent base_link, child base_imu, origin xyz=-0.07 -0.035 0.095 rpy=0 0 1.5707
- added joint base_link_to_base_laser: type fixed, parent base_link, child base_laser, origin xyz=0.095 -0.026 0.15 rpy=3.1415 0 1.5707

Commit message: added transformations from base_link to base_left_range, base_center_range and base_right_range

File: geduino/urdf/geduino.urdf (robot description, URDF)
Before this commit: robot geduino, 4 links, 3 joints
Links:
- added link base_center_range
- added link base_left_range
- added link base_right_range
Joints:
- added joint base_link_to_base_center_range: type fixed, parent base_link, child base_center_range, origin xyz=0.137 0 0.055 rpy=0 0 0
- added joint base_link_to_base_left_range: type fixed, parent base_link, child base_left_range, origin xyz=0.097 0.097 0.055 rpy=0 0 0.7853
- added joint base_link_to_base_right_range: type fixed, parent base_link, child base_right_range, origin xyz=0.097 -0.097 0.055 rpy=0 0 -0.7853

Commit message: refactored packages, moved configuration and launch files and some small fixes

File: geduino/urdf/geduino.urdf (robot description, URDF)
Before this commit: robot geduino, 7 links, 6 joints
Links:
- removed link base_camera
Joints:
- removed joint base_link_to_base_camera

Commit message: updated to new Geduino hardware

File: geduino/urdf/geduino.urdf (robot description, URDF)
Before this commit: robot geduino, 6 links, 5 joints
Links:
- removed link base_imu
Joints:
- removed joint base_link_to_base_imu
- joint base_link_to_base_laser: origin xyz=0.095 -0.026 0.15 rpy=3.1415 0 1.5707 -> xyz=0.000 0.000 0.15 rpy=3.1415 0 1.5707

Commit message: Adjusted launch file for multi-machine runs, added RealSense camera

File: geduino/urdf/geduino.urdf (robot description, URDF)
Before this commit: robot geduino, 5 links, 4 joints
Links:
- added link camera_link; visual box size=0.008 0.130 0.020
Joints:
- added joint base_link_to_camera_link: type fixed, parent base_link, child camera_link, origin xyz=0.125 -0.045 0.13 rpy=0 0 0

Commit message: Fixed base_link -> camera_link transformation

File: geduino/urdf/geduino.urdf (robot description, URDF)
Before this commit: robot geduino, 6 links, 5 joints
Joints:
- joint base_link_to_camera_link: origin xyz=0.125 -0.045 0.13 rpy=0 0 0 -> xyz=0.155 -0.045 0.13 rpy=0 0 0

Commit message: Added IMU configuration to shield param and base_imu to URDF

File: geduino/urdf/geduino.urdf (robot description, URDF)
Before this commit: robot geduino, 6 links, 5 joints
Links:
- added link base_imu
Joints:
- added joint base_link_to_base_imu: type fixed, parent base_link, child base_imu, origin xyz=-0.120 -0.050 0.060 rpy=0 0 0

Commit message: Fixed base_link -> camera_link transformation

File: geduino/urdf/geduino.urdf (robot description, URDF)
Before this commit: robot geduino, 7 links, 6 joints
Joints:
- joint base_link_to_camera_link: origin xyz=0.155 -0.045 0.13 rpy=0 0 0 -> xyz=0.135 -0.025 0.13 rpy=0 0 0

Commit message: Fixed base_link -> camera_link tf for new camera support

File: geduino/urdf/geduino.urdf (robot description, URDF)
Before this commit: robot geduino, 7 links, 6 joints
Joints:
- joint base_link_to_camera_link: origin xyz=0.135 -0.025 0.13 rpy=0 0 0 -> xyz=0.110 -0.030 0.13 rpy=0 0 0
